File: 36v4v.sch (KiCad schematic (older format))
At the start: 47 parts, among them J1 Conn_01x03, J2 Conn_01x02, J3 Conn_01x02, J4 Conn_01x02, J5 Conn_01x02, J6 Conn_01x02, J7 Conn_01x02, U1 InnoSwitch3-CE, INN3162C, inS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

Commit message: Added ground/heatsink for Innoswitch. Added C14 as per Anil
Parts:
- added C14: 10u 400V, Capacitor_THT:CP_Radial_D10.0mm_P5.00mm, symbol Device:CP_Small
- U1: footprint footprints:INN3162C-H1XX -> footprints:INN3162C-H1XX_
Connections:
- net sink is gone; now on net Earth: U1.16 (S)
- net Earth: now also U1.17 (S), U1.18 (S), U1.19 (S)
- net at C2.1, C3.1, C7.2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: now also C14.2
- net at C3.2, R2.2, R3.1: now also C14.1
Changed lines of the file:
@@
 $EndComp
 Wire Wire Line
-	4775 1450 5175 1450
+	4775 1450 5025 1450
 Wire Wire Line
 	5175 1450 5175 1500
@@
 F 0 "U1" V 7922 4578 60  0000 L CNN
 F 1 "InnoSwitch3-CE, INN3162C, inSOP-24D" V 8028 4578 60  0001 L CNN
-F 2 "footprints:INN3162C-H1XX" H 7975 4590 60  0001 C CNN
+F 2 "footprints:INN3162C-H1XX_" H 7975 4590 60  0001 C CNN
 F 3 "" H 7175 4350 60  0000 C CNN
 F 4 "Power Integrations" H 7175 4350 50  0001 C CNN "MFG Name"
@@
 Wire Wire Line
 	5175 3950 5575 3950
+Wire Wire Line
+	4450 4725 5175 4725
+Wire Wire Line
+	5575 4050 5175 4050
+Connection ~ 5175 4050
+Wire Wire Line
+	5175 4050 5175 3950
+Wire Wire Line
+	5575 4150 5175 4150
+Wire Wire Line
+	5175 4050 5175 4150
+Connection ~ 5175 4150
+Wire Wire Line
+	5175 4150 5175 4250
+Wire Wire Line
+	5575 4250 5175 4250
+Connection ~ 5175 4250
+Wire Wire Line
+	5175 4250 5175 4725
+$Comp
+L Device:CP_Small C14
+U 1 1 5ED262CB
+P 5025 1550
+F 0 "C14" H 5075 1400 50  0000 L CNN
+F 1 "10u 400V" H 4900 1325 50  0000 L CNN
+F 2 "Capacitor_THT:CP_Radial_D10.0mm_P5.00mm" H 5025 1550 50  0001 C CNN
+F 3 "~" H 5025 1550 50  0001 C CNN
+F 4 "Kemet/Panasonic" H 5025 1550 50  0001 C CNN "MFG Name"
+F 5 "ESH106M450AH4AA/EEV-EB2G100SM" H 5025 1550 50  0001 C CNN "MFG Part Num"
+	1    5025 1550
+	-1   0    0    1
+$EndComp
+Connection ~ 5025 1450
+Wire Wire Line
+	5025 1450 5175 1450
+Wire Wire Line
+	5025 1650 5025 1675
+Wire Wire Line
+	5025 1675 4975 1675
+Wire Wire Line
+	4975 1675 4975 1775
 $EndSCHEMATC
